File: esc/esc.kicad_pcb (KiCad board)
At the start: 2 copper layers, 90 x 90 mm, 44 parts, among them J1 Conn_01x04, J2 Conn_01x04, J3 Conn_01x01, J4 Conn_01x01, J5 Conn_01x03, J6 Conn_01x02, J7 Conn_01x02, J8 Conn_01x02, Q1 FDS2734, Q2 FDS2734, Q3 FDS2734, Q4 FDS2734, Q5 FDS2734, Q6 FDS2734, U1 STM32F051C8Tx, U2 KA78M05_TO252, U3 REGULAR-7133-1, U4 IR2103, U5 IR2103, U6 IR2103

Commit message: ...
Parts:
- added C6: C, Capacitor_SMD:C_0603_1608Metric_Pad1.05x0.95mm_HandSolder, F.Cu at (166.3, 71.6)
- added J10: Conn_01x01, Connector_Pin:Pin_D1.4mm_L8.5mm_W2.8mm_FlatFork, F.Cu at (159.7, 108.0)
- added J11: Conn_01x01, Connector_Pin:Pin_D1.4mm_L8.5mm_W2.8mm_FlatFork, F.Cu at (158.4, 130.0)
- added J12: Conn_01x01, Connector_Pin:Pin_D1.4mm_L8.5mm_W2.8mm_FlatFork, F.Cu at (165.7, 76.0)
- added J9: Conn_01x02, Connector_PinSocket_2.54mm:PinSocket_1x02_P2.54mm_Vertical, F.Cu at (133.4, 55.5)
- C1: footprint Capacitor_SMD:C_0603_1608Metric -> Capacitor_SMD:C_0603_1608Metric_Pad1.05x0.95mm_HandSolder
- C2: footprint Capacitor_SMD:C_0603_1608Metric_Pad1.05x0.95mm_HandSolder -> Capacitor_SMD:C_0603_1608Metric
- J3: value Conn_01x01 -> Conn_01x04; footprint Connector_Pin:Pin_D1.4mm_L8.5mm_W2.8mm_FlatFork -> Connector_PinSocket_2.54mm:PinSocket_1x04_P2.54mm_Vertical
- J5: value Conn_01x03 -> Conn_01x01; footprint Connector_PinSocket_2.54mm:PinSocket_1x03_P2.54mm_Vertical -> Connector_Pin:Pin_D1.4mm_L8.5mm_W2.8mm_FlatFork
- J6: value Conn_01x02 -> Conn_01x03; footprint Connector_PinSocket_2.54mm:PinSocket_1x02_P2.54mm_Vertical -> Connector_PinSocket_2.54mm:PinSocket_1x03_P2.54mm_Vertical
- U4, U5, U6: footprint Package_SO:SO-8_5.3x6.2mm_P1.27mm -> Package_SO:SO-8_3.9x4.9mm_P1.27mm
- moved BT1 116.0 mm to (24.5, 24.4)
- moved Q4 103.9 mm to (151.4, 130.0)
- moved U5 102.3 mm to (143.1, 129.6)
- moved Q3 88.7 mm to (165.7, 129.7)
- moved C4 85.9 mm to (163.0, 103.7), turned to 180 degrees
- moved D3 77.5 mm to (164.5, 124.9)
- moved U4 68.4 mm to (140.1, 108.5)
- moved Q2 67.9 mm to (150.5, 108.3)
- moved C5 63.6 mm to (159.4, 124.8), turned to 180 degrees
- moved C3 55.7 mm to (153.9, 60.0)
- moved J3 53.6 mm to (151.7, 31.0)
- moved Q1 50.1 mm to (168.6, 108.2)
- moved R4 49.1 mm to (149.4, 57.8)
- moved U6 47.8 mm to (148.1, 75.9)
- moved Q6 46.6 mm to (158.7, 76.0)
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Connections:
- C1 pad 1: Net-(C1-Pad1) -> +3V3
- C1 pad 2: RCP -> GND
- C2 pad 1: V_SAMPLE -> Net-(C2-Pad1)
- C2 pad 2: GND -> RCP
- C3 pad 1: Net-(C3-Pad1) -> V_SAMPLE
- C3 pad 2: /BOUT -> GND
- C4 pad 2: /COUT -> /BOUT
- C5 pad 2: /AOUT -> /COUT
- D2 pad 1: Net-(C3-Pad1) -> Net-(C4-Pad1)
- D3 pad 1: Net-(C4-Pad1) -> Net-(C5-Pad1)
- D4 pad 1: Net-(C5-Pad1) -> Net-(C6-Pad1)
- J1 pad 1: +3V3 -> /PA12
- J1 pad 2: GND -> /CP-OUT
- J1 pad 3: /SWCLK -> /PA2
- J1 pad 4: /SWDIO -> /PA3
- J2 pad 3: /RXD -> /SWCLK
- J2 pad 4: /TXD -> /SWDIO
- J3 pad 1: VCC -> +3V3
- J4 pad 1: GND -> VCC
- J5 pad 1: Net-(C1-Pad1) -> GND
- J6 pad 1: AP -> Net-(C2-Pad1)
- J6 pad 2: AN -> +5V
- J7 pad 1: BP -> AP
- J7 pad 2: BN -> AN
- J8 pad 1: CP -> BP
- J8 pad 2: CN -> BN
- U1 pad 12: Net-(U1-Pad12) -> /PA2
- U1 pad 13: Net-(U1-Pad13) -> /PA3
- U1 pad 2: Net-(U1-Pad2) -> (no net)
- U1 pad 20: Net-(U1-Pad20) -> (no net)
- U1 pad 21: Net-(U1-Pad21) -> (no net)
- U1 pad 25: Net-(U1-Pad25) -> (no net)
- U1 pad 26: Net-(U1-Pad26) -> (no net)
- U1 pad 27: Net-(U1-Pad27) -> (no net)
- U1 pad 28: Net-(U1-Pad28) -> (no net)
- U1 pad 3: Net-(U1-Pad3) -> (no net)
- U1 pad 32: Net-(U1-Pad32) -> /CP-OUT
- U1 pad 33: Net-(U1-Pad33) -> /PA12
- U1 pad 35: Net-(U1-Pad35) -> (no net)
- U1 pad 36: Net-(U1-Pad36) -> (no net)
- U1 pad 39: Net-(U1-Pad39) -> (no net)
- U1 pad 4: Net-(U1-Pad4) -> (no net)
- U1 pad 40: Net-(U1-Pad40) -> (no net)
- U1 pad 41: Net-(U1-Pad41) -> (no net)
- U1 pad 45: Net-(U1-Pad45) -> (no net)
- U1 pad 46: Net-(U1-Pad46) -> (no net)
- U1 pad 5: Net-(U1-Pad5) -> (no net)
- U1 pad 6: Net-(U1-Pad6) -> (no net)
- U4 pad 8: Net-(C3-Pad1) -> Net-(C4-Pad1)
- U5 pad 8: Net-(C4-Pad1) -> Net-(C5-Pad1)
- U6 pad 8: Net-(C5-Pad1) -> Net-(C6-Pad1)

Commit message: 已打样
Parts:
- removed BT1: Battery_Cell, Battery:BatteryHolder_Keystone_103_1x20mm
- removed J10, J11, J12: Conn_01x01, Connector_Pin:Pin_D1.4mm_L8.5mm_W2.8mm_FlatFork
- C2: moved to B.Cu
- moved J5 127.6 mm to (26.2, 72.8)
- moved J3 123.7 mm to (28.2, 24.2), turned to 90 degrees
- moved J4 123.3 mm to (26.2, 92.9)
- moved U3 121.3 mm to (38.2, 62.2), turned to 180 degrees
- moved R9 118.9 mm to (52.0, 59.4), turned to 90 degrees
- moved R11 117.3 mm to (50.1, 59.4), turned to 90 degrees
- moved R10 114.1 mm to (55.8, 54.6), turned to 90 degrees
- moved R3 111.9 mm to (46.2, 57.1), turned to 90 degrees
- moved R8 108.0 mm to (57.7, 54.6), turned to 90 degrees
- moved R6 105.8 mm to (59.7, 54.6), turned to 90 degrees
- moved C3 104.7 mm to (49.5, 53.7)
- moved R12 103.6 mm to (53.9, 54.6), turned to 90 degrees
- moved R14 103.4 mm to (57.7, 59.4), turned to 90 degrees
- moved R5 103.3 mm to (59.7, 59.4), turned to 90 degrees
- moved C1 103.1 mm to (55.9, 43.6), turned to 90 degrees
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Connections:
- J1 pad 1: /PA12 -> /PB13
- J1 pad 2: /CP-OUT -> /PB14
- J1 pad 3: /PA2 -> /PB15
- J1 pad 4: /PA3 -> /CP-OUT
- J3 pad 1: +3V3 -> +5V
- U1 pad 1: Net-(BT1-Pad1) -> +3V3
- U1 pad 12: /PA2 -> (no net)
- U1 pad 13: /PA3 -> (no net)
- U1 pad 26: (no net) -> /PB13
- U1 pad 27: (no net) -> /PB14
- U1 pad 28: (no net) -> /PB15
- U1 pad 33: /PA12 -> (no net)
Routing:
- net VCC: track 0.00 -> 124.9 mm
- net +5V: track 0.00 -> 115.4 mm
- net +3V3: track 0.00 -> 77.0 mm, vias 0 -> 3
- net /COUT: track 0.00 -> 67.8 mm, vias 0 -> 22
- net GND: track 0.00 -> 63.7 mm, vias 0 -> 44
- net /BOUT: track 0.00 -> 58.9 mm, vias 0 -> 22
- net /AOUT: track 0.00 -> 51.9 mm, vias 0 -> 22
- net CP: track 0.00 -> 49.2 mm
- net CN: track 0.00 -> 45.6 mm, vias 0 -> 1
- net /RXD: track 0.00 -> 41.8 mm
- net /TXD: track 0.00 -> 39.8 mm
- net BP: track 0.00 -> 38.1 mm
- net BN: track 0.00 -> 33.8 mm, vias 0 -> 1
- net /PB13: track 0.00 -> 32.7 mm
- net Net-(Q3-Pad4): track 0.00 -> 30.5 mm
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- added copper zone on B.Cu, net /AOUT
- added copper zone on F.Cu, net /AOUT
- added copper zone on B.Cu, net /BOUT
- added copper zone on F.Cu, net /BOUT
- added copper zone on B.Cu, net /COUT
- added copper zone on F.Cu, net /COUT
- added copper zone on B.Cu, net GND
- added copper zone on F.Cu, net VCC
Other:
- board text added: "+"
- board text added: "+|GND | CLK | DIO"
- board text added: "+|GND | RXD | TXD"
- board text added: "-"
- board text added: "AN AP"
- board text added: "BN BP"
- board text added: "CN CP"
- board text added: "CP| PB15 | PB14 | PB13"
- board text added: "PB11"

Commit message: driverless motor
Parts:
- removed D3, D4: D, Diode_SMD:D_0603_1608Metric_Pad1.05x0.95mm_HandSolder
- removed U4, U5, U6: IR2103, Package_SO:SO-8_3.9x4.9mm_P1.27mm
- added C7: C, Capacitor_SMD:C_0603_1608Metric_Pad1.05x0.95mm_HandSolder, F.Cu at (59.9, 87.9)
- added C8: C, Capacitor_THT:CP_Radial_D14.0mm_P5.00mm, F.Cu at (97.4, 100.5)
- added J10: Conn_01x03, Connector_PinHeader_2.54mm:PinHeader_1x03_P2.54mm_Vertical, F.Cu at (24.1, 71.1)
- added J11: Conn_01x05, Connector_PinHeader_2.54mm:PinHeader_1x05_P2.54mm_Vertical, F.Cu at (23.3, 97.0)
- added J12: Conn_01x06, Connector_PinHeader_2.54mm:PinHeader_1x06_P2.54mm_Vertical, F.Cu at (31.2, 106.1)
- added Q7: 2N3055, Package_TO_SOT_SMD:SOT-23, F.Cu at (80.5, 29.2)
- added Q8: nfet, footprint:SOIC-8, F.Cu at (90.8, 39.5)
- added Q9: pfet, footprint:SOIC-8, F.Cu at (90.8, 31.4)
- added R15: 1K, Resistor_SMD:R_0603_1608Metric_Pad1.05x0.95mm_HandSolder, F.Cu at (32.9, 31.5)
- added R16: R, Resistor_SMD:R_0603_1608Metric_Pad1.05x0.95mm_HandSolder, F.Cu at (81.5, 79.3)
- added R17: 1K, Resistor_SMD:R_0805_2012Metric_Pad1.15x1.40mm_HandSolder, F.Cu at (81.2, 65.0)
- added R18: R, Resistor_SMD:R_0603_1608Metric_Pad1.05x0.95mm_HandSolder, F.Cu at (81.6, 56.6)
- added R19: 1K, Resistor_SMD:R_0805_2012Metric_Pad1.15x1.40mm_HandSolder, F.Cu at (81.2, 45.3)
- added R20: R, Resistor_SMD:R_0603_1608Metric_Pad1.05x0.95mm_HandSolder, F.Cu at (81.7, 37.1)
- added R21: 1K, Resistor_SMD:R_0805_2012Metric_Pad1.15x1.40mm_HandSolder, F.Cu at (81.2, 25.6)
- added R22: 10K, Resistor_SMD:R_0603_1608Metric_Pad1.05x0.95mm_HandSolder, F.Cu at (28.5, 71.0)
- C2: footprint Capacitor_SMD:C_0603_1608Metric -> Capacitor_SMD:C_0603_1608Metric_Pad1.05x0.95mm_HandSolder; moved to F.Cu
- C5, C6: footprint Capacitor_SMD:C_0603_1608Metric_Pad1.05x0.95mm_HandSolder -> Capacitor_SMD:C_0805_2012Metric_Pad1.15x1.40mm_HandSolder
- D1: footprint LED_THT:LED_D4.0mm -> LED_THT:LED_D3.0mm
- D2: value D -> LED; footprint Diode_SMD:D_0603_1608Metric_Pad1.05x0.95mm_HandSolder -> LED_THT:LED_D3.0mm
- J1, J2: value Conn_01x04 -> Conn_01x01; footprint Connector_PinSocket_2.54mm:PinSocket_1x04_P2.54mm_Vertical -> Connector_Pin:Pin_D1.4mm_L8.5mm_W2.8mm_FlatFork
- J3: value Conn_01x04 -> Conn_01x01; footprint Connector_PinSocket_2.54mm:PinSocket_1x04_P2.54mm_Vertical -> MountingHole:MountingHole_3.5mm_Pad
- J4, J5: footprint Connector_Pin:Pin_D1.4mm_L8.5mm_W2.8mm_FlatFork -> MountingHole:MountingHole_3.5mm_Pad
- J6: value Conn_01x03 -> Conn_01x02; footprint Connector_PinSocket_2.54mm:PinSocket_1x03_P2.54mm_Vertical -> Connector_PinHeader_2.54mm:PinHeader_1x02_P2.54mm_Vertical
- J7, J8: value Conn_01x02 -> Conn_01x04; footprint Connector_PinSocket_2.54mm:PinSocket_1x02_P2.54mm_Vertical -> Connector_PinHeader_2.54mm:PinHeader_1x04_P2.54mm_Vertical
- J9: value Conn_01x02 -> Conn_01x03; footprint Connector_PinSocket_2.54mm:PinSocket_1x02_P2.54mm_Vertical -> Connector_PinHeader_2.54mm:PinHeader_1x03_P2.54mm_Vertical
- Q1, Q4: value FDS2734 -> 2N3055; footprint Package_SO:SOIC-8_3.9x4.9mm_P1.27mm -> Package_TO_SOT_SMD:SOT-23
- Q2, Q5: value FDS2734 -> nfet; footprint Package_SO:SOIC-8_3.9x4.9mm_P1.27mm -> footprint:SOIC-8
- Q3, Q6: value FDS2734 -> pfet; footprint Package_SO:SOIC-8_3.9x4.9mm_P1.27mm -> footprint:SOIC-8
- R1: value 1k -> 10K
- R10: value 3k -> 10K
- R11, R14: value 20k -> 1K
- R12: value 1k -> 1K
- R13, R5, R7, R9: value 20k -> 10K
- R2: value 1K -> 3K; footprint Resistor_THT:R_Axial_DIN0204_L3.6mm_D1.6mm_P7.62mm_Horizontal -> Resistor_SMD:R_0603_1608Metric_Pad1.05x0.95mm_HandSolder
- R3: value 2K -> 10K; footprint Resistor_SMD:R_0805_2012Metric_Pad1.15x1.40mm_HandSolder -> Resistor_SMD:R_0603_1608Metric_Pad1.05x0.95mm_HandSolder
- R4: value 2K -> 3K; footprint Resistor_SMD:R_0805_2012Metric_Pad1.15x1.40mm_HandSolder -> Resistor_SMD:R_0603_1608Metric_Pad1.05x0.95mm_HandSolder
- R6, R8: value 3k -> 3K
- U1: footprint Package_QFP:LQFP-48_7x7mm_P0.5mm -> footprint:QFP-48_P0.5mm_W0.22
- U2: value KA78M05_TO252 -> L7805
- U3: footprint Package_TO_SOT_SMD:SOT-89-3_Handsoldering -> Package_TO_SOT_SMD:SOT-89-3
- moved J3 87.8 mm to (101.1, 73.1)
- moved J2 87.5 mm to (81.1, 106.0)
- moved J1 86.2 mm to (106.8, 106.3), turned to 90 degrees
- moved J4 84.3 mm to (101.1, 54.1), turned to 90 degrees
- moved J5 83.8 mm to (101.1, 35.1), turned to 90 degrees
- moved D2 83.1 mm to (33.5, 25.1), turned to 0 degrees
- moved J9 77.3 mm to (23.6, 81.8), turned to 0 degrees
- moved C5 71.5 mm to (59.0, 24.6), turned to 0 degrees
- moved J8 62.1 mm to (25.5, 44.4), turned to 0 degrees
- moved D1 59.8 mm to (24.5, 24.8), turned to 0 degrees
- moved J6 56.4 mm to (36.6, 35.9), turned to 0 degrees
- moved C2 52.1 mm to (50.3, 61.2), turned to 90 degrees
- moved C6 50.3 mm to (59.6, 35.5), turned to 0 degrees
- moved J7 49.6 mm to (24.7, 57.4), turned to 0 degrees
- moved U2 48.7 mm to (61.6, 30.5), turned to 0 degrees
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Connections:
- C2 pad 1: Net-(C2-Pad1) -> +3V3
- C2 pad 2: RCP -> GND
- C3 pad 1: V_SAMPLE -> +3V3
- C4 pad 1: Net-(C4-Pad1) -> +3V3
- C4 pad 2: /BOUT -> GND
- C5 pad 1: Net-(C5-Pad1) -> VCC
- C5 pad 2: /COUT -> GND
- C6 pad 1: Net-(C6-Pad1) -> +5V
- C6 pad 2: /AOUT -> GND
- D2 pad 1: Net-(C4-Pad1) -> GND
- D2 pad 2: VCC -> Net-(D2-Pad2)
- J1 pad 1: /PB13 -> VCC
- J2 pad 1: +3V3 -> GND
- J3 pad 1: +5V -> OUT_A
- J4 pad 1: VCC -> OUT_B
- J5 pad 1: GND -> OUT_C
- J6 pad 1: Net-(C2-Pad1) -> RESET
- J6 pad 2: +5V -> GND
- J7 pad 1: AP -> +5V
- J7 pad 2: AN -> GND
- J8 pad 1: BP -> TEST1
- J8 pad 2: BN -> TEST2
- J9 pad 1: CP -> TEST5
- J9 pad 2: CN -> TEST6
- Q1 pad 1: /BOUT -> AP
- Q1 pad 2: /BOUT -> GND
- Q1 pad 3: /BOUT -> Net-(Q1-Pad3)
- Q2 pad 5: /BOUT -> OUT_A
- Q2 pad 6: /BOUT -> OUT_A
- Q2 pad 7: /BOUT -> OUT_A
- Q2 pad 8: /BOUT -> OUT_A
- Q3 pad 1: /COUT -> VCC
- Q3 pad 2: /COUT -> VCC
- Q3 pad 3: /COUT -> VCC
- Q3 pad 4: Net-(Q3-Pad4) -> Net-(Q1-Pad3)
- Q3 pad 5: VCC -> OUT_A
- Q3 pad 6: VCC -> OUT_A
- Q3 pad 7: VCC -> OUT_A
- Q3 pad 8: VCC -> OUT_A
- Q4 pad 1: GND -> BP
- Q4 pad 3: GND -> Net-(Q4-Pad3)
- Q5 pad 1: /AOUT -> GND
- Q5 pad 2: /AOUT -> GND
- Q5 pad 3: /AOUT -> GND
- Q5 pad 5: VCC -> OUT_B
- Q5 pad 6: VCC -> OUT_B
- Q5 pad 7: VCC -> OUT_B
- Q5 pad 8: VCC -> OUT_B
- Q6 pad 1: GND -> VCC
- Q6 pad 2: GND -> VCC
- Q6 pad 3: GND -> VCC
- Q6 pad 4: Net-(Q6-Pad4) -> Net-(Q4-Pad3)
- Q6 pad 5: /AOUT -> OUT_B
- Q6 pad 6: /AOUT -> OUT_B
- Q6 pad 7: /AOUT -> OUT_B
- Q6 pad 8: /AOUT -> OUT_B
- R1 pad 1: Net-(R1-Pad1) -> V_SAMPLE
- R1 pad 2: +3V3 -> VCC
- R10 pad 1: Fa -> Fabc
- R10 pad 2: GND -> OUT_B
- R11 pad 1: /AOUT -> GND
- R12 pad 1: Fabc -> RESET
- R12 pad 2: GND -> +3V3
- R13 pad 1: /BOUT -> Fabc
- R13 pad 2: Fabc -> OUT_C
- R14 pad 1: /COUT -> Net-(D1-Pad2)
- R14 pad 2: Fabc -> LED1
- R2 pad 1: Net-(D1-Pad2) -> GND
- R2 pad 2: /LED -> V_SAMPLE
- R3 pad 1: VCC -> Fa
- R3 pad 2: V_SAMPLE -> OUT_A
- R4 pad 1: V_SAMPLE -> GND
- R4 pad 2: GND -> Fa
- R5 pad 1: /COUT -> Fb
- R5 pad 2: Fc -> OUT_B
- R6 pad 1: Fc -> GND
- R6 pad 2: GND -> Fb
- R7 pad 1: /BOUT -> Fc
- R7 pad 2: Fb -> OUT_C
- R8 pad 1: Fb -> GND
- R8 pad 2: GND -> Fc
- R9 pad 1: /AOUT -> Fabc
- R9 pad 2: Fa -> OUT_A
- U1 pad 12: (no net) -> Net-(U1-Pad12)
- U1 pad 13: (no net) -> Net-(U1-Pad13)
- U1 pad 17: AP -> CP
- U1 pad 18: BP -> LED2
- U1 pad 19: CP -> LED1
- U1 pad 2: (no net) -> Net-(U1-Pad2)
- U1 pad 20: (no net) -> Net-(U1-Pad20)
- U1 pad 21: (no net) -> TEST3
- U1 pad 22: /LED -> TEST4
- U1 pad 25: (no net) -> TEST5
- U1 pad 26: /PB13 -> TEST6
- U1 pad 27: /PB14 -> AN
- U1 pad 28: /PB15 -> AP
- U1 pad 29: AN -> CN
- U1 pad 3: (no net) -> Net-(U1-Pad3)
- U1 pad 30: BN -> BP
- U1 pad 31: CN -> BN
- U1 pad 32: /CP-OUT -> CPOUT
- U1 pad 33: (no net) -> Net-(U1-Pad33)
- U1 pad 34: /SWDIO -> SWDIO
- U1 pad 35: (no net) -> Net-(U1-Pad35)
- U1 pad 36: (no net) -> Net-(U1-Pad36)
- U1 pad 37: /SWCLK -> SWCLK
- U1 pad 39: (no net) -> Net-(U1-Pad39)
- U1 pad 4: (no net) -> Net-(U1-Pad4)
- U1 pad 40: (no net) -> Net-(U1-Pad40)
- U1 pad 41: (no net) -> Net-(U1-Pad41)
- U1 pad 42: /TXD -> TXD
- U1 pad 43: /RXD -> RXD
- U1 pad 45: (no net) -> TEST1
- U1 pad 46: (no net) -> TEST2
- U1 pad 5: (no net) -> Net-(U1-Pad5)
- U1 pad 6: (no net) -> Net-(U1-Pad6)
- U1 pad 7: Net-(R1-Pad1) -> RESET
Routing:
- net +5V: track 115.4 -> 7.34 mm
- net +3V3: track 77.0 -> 0.00 mm, vias 3 -> 0
- net /COUT: track 67.8 -> 0.00 mm, vias 22 -> 0
- net /BOUT: track 58.9 -> 0.00 mm, vias 22 -> 0
- net /AOUT: track 51.9 -> 0.00 mm, vias 22 -> 0
- net CP: track 49.2 -> 0.00 mm
- net GND: track 63.7 -> 15.0 mm, vias 44 -> 0
- net CN: track 45.6 -> 0.00 mm, vias 1 -> 0
- net /RXD: track 41.8 -> 0.00 mm
- net /TXD: track 39.8 -> 0.00 mm
- net BP: track 38.1 -> 0.00 mm
- net BN: track 33.8 -> 0.00 mm, vias 1 -> 0
- net /PB13: track 32.7 -> 0.00 mm
- net Net-(Q3-Pad4): track 30.5 -> 0.00 mm
- net Net-(Q5-Pad4): track 30.4 -> 0.00 mm
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- added copper zone on F.Cu, net OUT_A
- removed copper zone on B.Cu, net /AOUT
- removed copper zone on F.Cu, net /AOUT
- removed copper zone on B.Cu, net /BOUT
- removed copper zone on F.Cu, net /BOUT
- removed copper zone on B.Cu, net /COUT
- removed copper zone on F.Cu, net /COUT
- removed copper zone on B.Cu, net GND
- removed copper zone on F.Cu, net VCC
Other:
- board text removed: "+"
- board text removed: "+|GND | CLK | DIO"
- board text removed: "+|GND | RXD | TXD"
- board text removed: "-"
- board text removed: "AN AP"
- board text removed: "BN BP"
- board text removed: "CN CP"
- board text removed: "CP| PB15 | PB14 | PB13"
- board text removed: "PB11"

Commit message: ...
Parts:
- J1, J2: footprint Connector_Pin:Pin_D1.4mm_L8.5mm_W2.8mm_FlatFork -> MountingHole:MountingHole_2.5mm_Pad
- J3, J4, J5: footprint MountingHole:MountingHole_3.5mm_Pad -> MountingHole:MountingHole_2.5mm_Pad
- moved J2 2.88 mm to (78.7, 104.4)
- moved J1 2.84 mm to (104.7, 104.4)
- moved C8 2.64 mm to (94.8, 99.9)
Routing:
- net VCC: track 132.2 -> 0.00 mm
- added copper zone on F.Cu, net OUT_B
- added copper zone on F.Cu, net OUT_C

Commit message: imcomplete yet
Parts:
- J1: value Conn_01x01 -> 12V
- J10: value Conn_01x03 -> GND V5 RCP
- J11: value Conn_01x05 -> 5V GND DIO CLK
- J12: value Conn_01x06 -> AP AN BP BN CP CN
- J2: value Conn_01x01 -> GND
- J3: value Conn_01x01 -> A
- J4: value Conn_01x01 -> B
- J5: value Conn_01x01 -> C
- J6: value Conn_01x02 -> RESET
- J7: value Conn_01x04 -> V5 GND TXD RXD
- J8: value Conn_01x04 -> T4 T3 T2 T1
- J9: value Conn_01x03 -> CP T6 T5
- R22: value 10K -> 1K
- moved J11 86.3 mm to (68.8, 23.7), turned to 270 degrees
- moved J8 49.1 mm to (44.6, 89.6), turned to 180 degrees
- moved R12 40.9 mm to (49.7, 71.1), turned to 90 degrees
- moved J7 38.9 mm to (44.3, 23.7), turned to 90 degrees
- moved D1 38.1 mm to (60.2, 38.2), turned to 180 degrees
- moved J10 37.7 mm to (44.6, 39.5), turned to 180 degrees
- moved R22 37.4 mm to (50.1, 40.3), turned to 90 degrees
- moved J6 37.0 mm to (44.8, 72.0), turned to 180 degrees
- moved C5 36.2 mm to (95.2, 24.4), turned to 180 degrees
- moved D2 34.9 mm to (65.9, 38.2), turned to 180 degrees
- moved R14 31.9 mm to (58.6, 33.2), turned to 0 degrees
- moved R15 31.3 mm to (64.2, 33.2)
- moved J9 29.9 mm to (44.6, 103.1), turned to 180 degrees
- moved C1 29.0 mm to (76.8, 35.9)
- moved U3 28.6 mm to (80.9, 36.0)
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Connections:
- J11 pad 4: Net-(J11-Pad4) -> GND
- U1 pad 12: Net-(U1-Pad12) -> LED1
- U1 pad 13: Net-(U1-Pad13) -> LED2
- U1 pad 17: CP -> TEST4
- U1 pad 18: LED2 -> AN
- U1 pad 19: LED1 -> AP
- U1 pad 20: Net-(U1-Pad20) -> BN
- U1 pad 21: TEST3 -> BP
- U1 pad 22: TEST4 -> CN
- U1 pad 25: TEST5 -> CP
- U1 pad 27: AN -> Net-(U1-Pad27)
- U1 pad 28: AP -> Net-(U1-Pad28)
- U1 pad 29: CN -> TEST3
- U1 pad 30: BP -> TEST2
- U1 pad 31: BN -> TEST1
- U1 pad 45: TEST1 -> Net-(U1-Pad45)
- U1 pad 46: TEST2 -> TEST5
Routing:
- net VCC: track 0.00 -> 131.2 mm
- net +5V: track 7.34 -> 69.5 mm
- net OUT_C: track 0.00 -> 50.5 mm, vias 0 -> 2
- net OUT_B: track 0.00 -> 39.0 mm
- net OUT_A: track 0.00 -> 37.1 mm
- net GND: track 15.0 -> 52.0 mm, vias 0 -> 23
- net AN: track 0.00 -> 35.6 mm, vias 0 -> 2
- net +3V3: track 0.00 -> 34.9 mm
- net AP: track 0.00 -> 29.9 mm, vias 0 -> 2
- net BN: track 0.00 -> 25.4 mm, vias 0 -> 2
- net CP: track 0.00 -> 22.5 mm
- net CN: track 0.00 -> 21.4 mm
- net Fc: track 0.00 -> 19.6 mm
- net Fa: track 0.00 -> 19.3 mm
- net BP: track 0.00 -> 17.8 mm
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- added copper zone on B.Cu, net GND
- added copper zone on F.Cu, net GND
- added copper zone on F.Cu, net VCC
Other:
- board size 90 x 90 mm -> 70 x 90 mm

Commit message: not done yet
Parts:
- added J13: AN, footprint:CONN1-DR1.0-W2.0, F.Cu at (73.4, 84.1)
- added J14: BP, footprint:CONN1-DR1.0-W2.0, F.Cu at (75.3, 63.8)
- added J15: BN, footprint:CONN1-DR1.0-W2.0, F.Cu at (75.3, 66.9)
- added J16: CP, footprint:CONN1-DR1.0-W2.0, F.Cu at (74.5, 45.5)
- added J17: CN, footprint:CONN1-DR1.0-W2.0, F.Cu at (74.9, 51.8)
- J10: value GND V5 RCP -> RCP V5 GND
- J11: value 5V GND DIO CLK -> CLK DIO G G 5V
- J12: value AP AN BP BN CP CN -> AP; footprint Connector_PinHeader_2.54mm:PinHeader_1x06_P2.54mm_Vertical -> footprint:CONN1-DR1.0-W2.0
- J7: value V5 GND TXD RXD -> V5 GND RXD TXD
- J8: value T4 T3 T2 T1 -> T1 T2 T3 T4; footprint Connector_PinHeader_2.54mm:PinHeader_1x04_P2.54mm_Vertical -> footprint:CONN4-P2.54-DR1.0-W1.5
- J9: value CP T6 T5 -> T5 T6 CP
- moved J9 49.1 mm to (44.8, 54.0)
- moved J12 31.3 mm to (74.6, 80.2)
- moved J8 15.8 mm to (44.9, 73.8), turned to 90 degrees
- moved R15 12.5 mm to (54.5, 41.1)
- moved J11 10.5 mm to (58.3, 23.7), turned to 90 degrees
- moved D2 9.76 mm to (56.2, 36.9)
- moved R14 8.26 mm to (60.9, 41.1)
- moved J6 7.45 mm to (52.2, 71.2), turned to 90 degrees
- moved R22 5.55 mm to (45.7, 43.7)
- moved R12 3.84 mm to (50.9, 67.4)
- moved D1 2.68 mm to (62.6, 36.9)
Connections:
- J7 pad 3: TXD -> RXD
- J7 pad 4: RXD -> TXD
- U1 pad 12: LED1 -> Net-(U1-Pad12)
- U1 pad 13: LED2 -> Net-(U1-Pad13)
- U1 pad 17: TEST4 -> Net-(U1-Pad17)
- U1 pad 2: Net-(U1-Pad2) -> TEST4
- U1 pad 26: TEST6 -> LED1
- U1 pad 27: Net-(U1-Pad27) -> LED2
- U1 pad 45: Net-(U1-Pad45) -> TEST6
Routing:
- net +3V3: track 34.9 -> 141.1 mm
- net SWDIO: track 0.00 -> 45.5 mm
- net SWCLK: track 0.00 -> 41.7 mm
- net TXD: track 0.00 -> 39.3 mm
- net RXD: track 0.00 -> 39.2 mm
- net TEST1: track 0.00 -> 36.1 mm, vias 0 -> 1
- net TEST2: track 0.00 -> 33.5 mm, vias 0 -> 1
- net GND: track 52.0 -> 84.9 mm, vias 23 -> 27
- net TEST3: track 0.00 -> 31.1 mm, vias 0 -> 1
- net V_SAMPLE: track 4.28 -> 30.0 mm, vias 0 -> 2
- net RCP: track 0.00 -> 24.1 mm, vias 0 -> 2
- net Fabc: track 6.16 -> 23.5 mm, vias 0 -> 2
- net LED2: track 0.00 -> 17.0 mm
- net TEST6: track 0.00 -> 15.5 mm
- net CPOUT: track 0.00 -> 15.4 mm, vias 0 -> 1
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Other:
- net class power added: clearance 0.2, trace_width 0.4, via_dia 0.8, via_drill 0.4

Commit message: incomplete
Parts:
- removed J15: BN, footprint:CONN1-DR1.0-W2.0
- removed J16: CP, footprint:CONN1-DR1.0-W2.0
- removed J17: CN, footprint:CONN1-DR1.0-W2.0
- C1: footprint Capacitor_SMD:C_0603_1608Metric_Pad1.05x0.95mm_HandSolder -> Capacitor_THT:CP_Radial_D14.0mm_P5.00mm
- C2: footprint Capacitor_SMD:C_0603_1608Metric_Pad1.05x0.95mm_HandSolder -> Capacitor_SMD:C_0603_1608Metric_Pad1.08x0.95mm_HandSolder
- C3, C4: footprint Capacitor_SMD:C_0603_1608Metric_Pad1.05x0.95mm_HandSolder -> Capacitor_SMD:C_0603_1608Metric
- C5, C6: footprint Capacitor_SMD:C_0805_2012Metric_Pad1.15x1.40mm_HandSolder -> Capacitor_SMD:C_0603_1608Metric
- C7: footprint Capacitor_SMD:C_0603_1608Metric_Pad1.05x0.95mm_HandSolder -> Capacitor_SMD:C_0805_2012Metric
- C8: footprint Capacitor_THT:CP_Radial_D14.0mm_P5.00mm -> Capacitor_SMD:C_0805_2012Metric
- J10, J9: footprint Connector_PinHeader_2.54mm:PinHeader_1x03_P2.54mm_Vertical -> footprint:CONN3-P2.54-DR1.0-W1.5
- J11: value CLK DIO G G 5V -> AN AP; footprint Connector_PinHeader_2.54mm:PinHeader_1x05_P2.54mm_Vertical -> footprint:CONN2-P2.54-DR1.0-W1.3
- J12: value AP -> BN BP; footprint footprint:CONN1-DR1.0-W2.0 -> footprint:CONN2-P2.54-DR1.0-W1.3
- J13: value AN -> CN CP; footprint footprint:CONN1-DR1.0-W2.0 -> footprint:CONN2-P2.54-DR1.0-W1.3
- J14: value BP -> CLK DIO GND 5V; footprint footprint:CONN1-DR1.0-W2.0 -> footprint:CONN4-P2.54-DR1.0-W1.5
- J6: footprint Connector_PinHeader_2.54mm:PinHeader_1x02_P2.54mm_Vertical -> footprint:CONN2-P2.54-DR1.0-W1.3
- J7: footprint Connector_PinHeader_2.54mm:PinHeader_1x04_P2.54mm_Vertical -> footprint:CONN4-P2.54-DR1.0-W1.5
- R1: value 10K -> Rcc; footprint Resistor_SMD:R_0603_1608Metric_Pad1.05x0.95mm_HandSolder -> Resistor_SMD:R_0603_1608Metric_Pad0.98x0.95mm_HandSolder
- R10, R11, R12, R13, R14, R15, R3, R4, R5, R6, R7, R8, R9: footprint Resistor_SMD:R_0603_1608Metric_Pad1.05x0.95mm_HandSolder -> Resistor_SMD:R_0603_1608Metric_Pad0.98x0.95mm_HandSolder
- R16: value R -> 1K; footprint Resistor_SMD:R_0603_1608Metric_Pad1.05x0.95mm_HandSolder -> Resistor_SMD:R_0603_1608Metric_Pad0.98x0.95mm_HandSolder
- R17, R19, R21: value 1K -> R; footprint Resistor_SMD:R_0805_2012Metric_Pad1.15x1.40mm_HandSolder -> Resistor_SMD:R_0603_1608Metric_Pad0.98x0.95mm_HandSolder
- R18, R20: value R -> 1K; footprint Resistor_SMD:R_0603_1608Metric_Pad1.05x0.95mm_HandSolder -> Resistor_SMD:R_0805_2012Metric_Pad1.20x1.40mm_HandSolder
- R2: value 3K -> Rss; footprint Resistor_SMD:R_0603_1608Metric_Pad1.05x0.95mm_HandSolder -> Resistor_SMD:R_0603_1608Metric_Pad0.98x0.95mm_HandSolder
- R22: footprint Resistor_SMD:R_0603_1608Metric_Pad1.05x0.95mm_HandSolder -> Resistor_SMD:R_0805_2012Metric_Pad1.20x1.40mm_HandSolder
- moved R14 102.6 mm to (-10.9, 114.3)
- moved U2 95.7 mm to (40.0, 111.8), turned to 270 degrees
- moved D2 88.5 mm to (6.38, 110.1), turned to 0 degrees
- moved J10 87.8 mm to (-6.20, 111.0), turned to 0 degrees
- moved D1 80.8 mm to (16.0, 102.9), turned to 0 degrees
- moved U3 80.1 mm to (37.7, 103.4), turned to 270 degrees
- moved C5 76.9 mm to (38.9, 76.7), turned to 90 degrees
- moved C1 74.6 mm to (84.4, 110.1), turned to 180 degrees
- moved R16 70.9 mm to (12.8, 110.0), turned to 0 degrees
- moved J7 70.1 mm to (33.7, 93.0)
- moved J11 64.8 mm to (64.5, 88.2), turned to 270 degrees
- moved J9 64.4 mm to (-1.49, 98.7), turned to 0 degrees
- moved C8 60.2 mm to (34.2, 109.8), turned to 270 degrees
- moved J8 57.0 mm to (-4.02, 103.0), turned to 0 degrees
- moved R15 56.7 mm to (27.2, 90.7)
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Connections:
- C1 pad 1: +3V3 -> VCC
- C2 pad 1: +3V3 -> V_SAMPLE
- C5 pad 1: VCC -> +3V3
- C6 pad 1: +5V -> +3V3
- C7 pad 1: V_SAMPLE -> VCC
- C8 pad 1: VCC -> +5V
- J11 pad 1: SWCLK -> AP
- J11 pad 2: SWDIO -> AN
- J12 pad 1: AP -> BP
- J13 pad 1: AN -> CP
- J14 pad 1: BP -> +5V
- R16 pad 1: Net-(Q2-Pad4) -> RCP
- R16 pad 2: AN -> Net-(J10-Pad1)
- R17 pad 1: VCC -> Net-(Q2-Pad4)
- R17 pad 2: Net-(Q1-Pad3) -> AN
- R18 pad 1: Net-(Q5-Pad4) -> VCC
- R18 pad 2: BN -> Net-(Q1-Pad3)
- R19 pad 1: VCC -> Net-(Q5-Pad4)
- R19 pad 2: Net-(Q4-Pad3) -> BN
- R20 pad 1: Net-(Q8-Pad4) -> VCC
- R20 pad 2: CN -> Net-(Q4-Pad3)
- R21 pad 1: VCC -> Net-(Q8-Pad4)
- R21 pad 2: Net-(Q7-Pad3) -> CN
- R22 pad 1: RCP -> VCC
- R22 pad 2: Net-(J10-Pad1) -> Net-(Q7-Pad3)
Routing:
- net +3V3: track 141.1 -> 63.5 mm, vias 0 -> 3
- net TXD: track 39.3 -> 0.00 mm
- net RXD: track 39.2 -> 0.00 mm
- net TEST1: track 36.1 -> 0.00 mm, vias 1 -> 0
- net TEST2: track 33.5 -> 0.00 mm, vias 1 -> 0
- net TEST3: track 31.1 -> 0.00 mm, vias 1 -> 0
- net RCP: track 24.1 -> 0.00 mm, vias 2 -> 0
- net GND: track 84.9 -> 63.4 mm, vias 27 -> 24
- net SWDIO: track 45.5 -> 63.4 mm, vias 0 -> 2
- net LED2: track 17.0 -> 0.00 mm
- net TEST6: track 15.5 -> 0.00 mm
- net CPOUT: track 15.4 -> 0.00 mm, vias 1 -> 0
- net LED1: track 15.0 -> 0.00 mm
- net VCC: track 140.0 -> 125.0 mm
- net +5V: track 66.6 -> 51.9 mm, vias 1 -> 0
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