File: esc/esc.kicad_pcb (KiCad board)
At the start: 2 copper layers, 70 x 90 mm, 58 parts, among them J1 12V, J10 RCP V5 GND, J11 AN AP, J12 BN BP, J13 CN CP, J14 CLK DIO GND 5V, J2 GND, J3 A, J4 B, J5 C, J6 RESET, J7 V5 GND RXD TXD, J8 T1 T2 T3 T4, J9 T5 T6 CP, Q1 2N3055, Q2 nfet, Q3 pfet, Q4 2N3055, Q5 nfet, Q6 pfet, Q7 2N3055, Q8 nfet, Q9 pfet, U1 STM32F051C8Tx, U2 L7805, U3 REGULAR-7133-1

Commit message: ...
Parts:
- moved R14 98.5 mm to (61.6, 47.7), turned to 180 degrees
- moved J8 84.5 mm to (44.2, 33.6)
- moved D2 82.4 mm to (54.0, 42.8)
- moved D1 74.5 mm to (60.0, 42.8)
- moved J9 67.3 mm to (33.7, 41.3), turned to 90 degrees
- moved J14 61.9 mm to (33.7, 54.7), turned to 270 degrees
- moved J10 59.0 mm to (33.7, 67.5), turned to 90 degrees
- moved R15 50.4 mm to (55.1, 48.7)
- moved R16 42.8 mm to (34.6, 73.2), turned to 180 degrees
Connections:
- U1 pad 2: TEST4 -> Net-(U1-Pad2)
- U1 pad 28: Net-(U1-Pad28) -> TEST4
- U1 pad 35: Net-(U1-Pad35) -> TEST6
- U1 pad 36: Net-(U1-Pad36) -> TEST5
- U1 pad 45: TEST6 -> Net-(U1-Pad45)
- U1 pad 46: TEST5 -> Net-(U1-Pad46)
Routing:
- net CPOUT: track 0.00 -> 41.4 mm
- net TEST1: track 0.00 -> 38.6 mm
- net SWDIO: track 63.4 -> 25.3 mm, vias 2 -> 1
- net TEST2: track 0.00 -> 37.8 mm
- net TEST6: track 0.00 -> 37.5 mm
- net TEST3: track 0.00 -> 36.9 mm
- net TEST4: track 0.00 -> 36.1 mm
- net TEST5: track 0.00 -> 35.4 mm
- net GND: track 63.4 -> 95.9 mm
- net SWCLK: track 49.8 -> 19.8 mm, vias 2 -> 0
- net RXD: track 0.00 -> 25.4 mm
- net TXD: track 0.00 -> 22.7 mm
- net +5V: track 51.9 -> 71.8 mm
- net RCP: track 0.00 -> 8.20 mm
- net Net-(J10-Pad1): track 0.00 -> 3.12 mm
