File: esc/esc.kicad_pcb (KiCad board)
At the start: 2 copper layers, 70 x 90 mm, 58 parts, among them J1 12V, J10 RCP V5 GND, J11 AN AP, J12 BN BP, J13 CN CP, J14 CLK DIO GND 5V, J2 GND, J3 A, J4 B, J5 C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

Commit message: ...
Parts:
- moved D1 30.3 mm to (89.4, 35.4)
- moved R14 26.2 mm to (85.6, 37.3)
- moved D2 23.6 mm to (76.4, 35.4)
- moved R15 20.4 mm to (72.0, 37.3), turned to 180 degrees
- moved J8 20.3 mm to (64.5, 33.6)
- moved J13 4.00 mm to (64.2, 60.9)
Routing:
- net LED1: track 0.00 -> 64.8 mm
- net LED2: track 0.00 -> 51.7 mm
- net TEST4: track 36.1 -> 51.1 mm
- net TEST3: track 36.9 -> 49.1 mm
- net TEST2: track 37.8 -> 47.2 mm
- net Net-(D2-Pad2): track 0.00 -> 6.86 mm
- net TEST1: track 38.6 -> 45.2 mm
- net Net-(D1-Pad2): track 0.00 -> 6.15 mm
- net OUT_C: track 52.1 -> 49.3 mm
- net CN: track 29.4 -> 28.1 mm
- net CP: track 32.9 -> 32.1 mm
- net BP: track 21.3 -> 20.7 mm, vias 1 -> 0
- net BN: track 21.5 -> 21.1 mm, vias 1 -> 0

Commit message: almost done
Parts:
- moved J10 31.8 mm to (34.0, 35.7)
- moved R16 31.1 mm to (35.2, 42.1)
- moved C8 17.3 mm to (51.3, 107.0)
- moved J9 16.2 mm to (48.1, 33.8), turned to 0 degrees
- moved R12 12.6 mm to (39.7, 70.3)
- moved J6 12.5 mm to (43.0, 71.6)
- moved C6 11.8 mm to (55.9, 58.8)
- moved U1 11.8 mm to (47.1, 61.9)
- moved C2 11.8 mm to (48.7, 90.9)
- moved R1 11.8 mm to (54.6, 90.9)
- moved R10 11.8 mm to (54.6, 88.3)
- moved R11 11.8 mm to (48.8, 85.7)
- moved R13 11.8 mm to (54.6, 83.0)
- moved R2 11.8 mm to (48.8, 88.3)
- moved R3 11.8 mm to (54.6, 80.4)
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Routing:
- net +5V: track 71.8 -> 103.8 mm
- net +3V3: track 63.4 -> 88.8 mm
- net VCC: track 125.0 -> 103.8 mm
- net CPOUT: track 41.4 -> 25.6 mm
- net RCP: track 8.20 -> 21.5 mm, vias 0 -> 2
- net TEST6: track 37.5 -> 25.2 mm
- net TEST5: track 35.4 -> 24.3 mm
- net TEST2: track 47.2 -> 36.5 mm
- net TEST1: track 45.2 -> 34.6 mm
- net TEST4: track 51.1 -> 40.4 mm
- net TEST3: track 49.1 -> 38.5 mm
- net LED2: track 51.7 -> 41.1 mm
- net LED1: track 64.8 -> 54.4 mm
- net SWDIO: track 25.3 -> 15.0 mm, vias 1 -> 0
- net RXD: track 25.4 -> 34.9 mm
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
Commit message: confirm
Parts:
- J7: value V5 GND RXD TXD -> V5 GND RX TX
Routing:
- net VCC: track 103.8 -> 99.4 mm
- net Net-(Q5-Pad4): track 15.7 -> 12.4 mm
- net OUT_C: track 45.4 -> 44.8 mm
