File: m48/m48.kicad_pcb (KiCad board)
At the start: 2 copper layers, 70 x 90 mm, 51 parts, among them J10 CN CP, J11 Conn_01x06, J3 A, J4 B, J5 C, J6 T1 T2 T3 T4 T5, J7 RCP V5 GND, J8 AN AP, J9 BN BP, Q1 2N3055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

Commit message: default width 0.3mm
Parts:
- moved C2 1.09 mm to (83.6, 59.0)
Routing:
- net AN: track 0.00 -> 51.5 mm
- net Fabc: track 7.25 -> 40.9 mm
- net AP: track 0.00 -> 32.8 mm
- net Fb: track 7.56 -> 33.2 mm
- net BN: track 0.00 -> 22.5 mm
- net Fc: track 7.42 -> 27.2 mm, vias 0 -> 2
- net VCC: track 17.3 -> 0.00 mm
- net +5V: track 0.00 -> 8.33 mm
- net GND: track 28.5 -> 34.9 mm
- net CP: track 24.4 -> 19.0 mm
- net BP: track 19.2 -> 14.1 mm
- net Net-(U1-Pad8): track 0.00 -> 4.88 mm
- net CN: track 22.0 -> 26.4 mm
- net Net-(U1-Pad7): track 0.00 -> 4.38 mm
Other:
- net class Default: trace_width 0.25 -> 0.3

Commit message: working
Parts:
- moved C4 47.4 mm to (95.3, 52.0), turned to 270 degrees
- moved R2 44.4 mm to (95.3, 48.0), turned to 90 degrees
- moved R3 41.6 mm to (92.3, 52.0), turned to 90 degrees
- moved J10 33.1 mm to (61.0, 76.1), turned to 180 degrees
- moved R14 22.1 mm to (71.6, 34.7)
- moved J9 21.5 mm to (75.2, 76.1), turned to 180 degrees
- moved J11 19.1 mm to (80.9, 33.5), turned to 90 degrees
- moved J8 18.3 mm to (89.5, 76.1), turned to 180 degrees
- moved Q7 12.7 mm to (58.8, 85.8)
- moved R13 11.6 mm to (58.2, 34.7)
- moved Q1 11.4 mm to (87.3, 85.8)
- moved Q4 11.3 mm to (73.0, 85.8)
- moved D2 11.1 mm to (64.4, 34.7)
- moved R17 10.3 mm to (87.3, 108.6)
- moved R19 10.3 mm to (73.0, 108.6)
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- renumbered + to J1, - to J2
Connections:
- J11 pad 3: MOSI -> SCK
- J11 pad 5: SCK -> MOSI
- U1 pad 11: Fb -> Fc
- U1 pad 19: Fc -> Fb
Routing:
- net +5V: track 8.33 -> 150.3 mm, vias 0 -> 1
- net VCC: track 0.00 -> 75.0 mm
- net OUT_A: track 0.00 -> 63.7 mm, vias 0 -> 12
- net OUT_C: track 0.00 -> 57.7 mm, vias 0 -> 10
- net TEST4: track 0.00 -> 56.8 mm, vias 0 -> 1
- net OUT_B: track 0.00 -> 50.9 mm, vias 0 -> 12
- net TEST3: track 0.00 -> 48.6 mm, vias 0 -> 1
- net RESET: track 0.00 -> 39.6 mm, vias 0 -> 2
- net LED1: track 0.00 -> 39.4 mm, vias 0 -> 2
- net Net-(Q1-Pad3): track 0.00 -> 32.0 mm
- net Net-(Q7-Pad3): track 0.00 -> 32.0 mm
- net CP: track 19.0 -> 50.8 mm
- net Net-(Q4-Pad3): track 0.00 -> 31.5 mm
- net LED2: track 0.00 -> 24.1 mm, vias 0 -> 2
- net BP: track 14.1 -> 37.5 mm
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
Commit message: issued
Parts:
- moved D2 15.1 mm to (49.3, 35.9)
- moved R14 15.1 mm to (56.5, 35.9)
- moved R13 12.8 mm to (71.0, 35.8)
- moved D1 12.8 mm to (63.9, 35.8)
- moved C6 12.1 mm to (37.7, 63.8), turned to 0 degrees
- moved C5 8.41 mm to (51.9, 91.5)
- moved R2 1.35 mm to (96.2, 49.0), turned to 0 degrees
Connections:
- U1 pad 13: TEST1 -> LED1
- U1 pad 14: TEST2 -> LED2
- U1 pad 23: TEST3 -> TEST5
- U1 pad 25: LED2 -> TEST3
- U1 pad 26: LED1 -> TEST2
- U1 pad 27: TEST5 -> TEST1
Routing:
- net VCC: track 75.0 -> 157.9 mm, vias 0 -> 2
- net TEST5: track 0.00 -> 53.9 mm, vias 0 -> 2
- net TEST2: track 0.00 -> 51.1 mm, vias 0 -> 2
- net TEST1: track 0.00 -> 51.1 mm, vias 0 -> 2
- net RCP: track 0.00 -> 45.7 mm, vias 0 -> 4
- net LED1: track 39.4 -> 17.3 mm
- net Net-(J7-Pad1): track 0.00 -> 7.43 mm
- net TEST4: track 56.8 -> 51.6 mm, vias 1 -> 2
- net LED2: track 24.1 -> 29.1 mm
- net TEST3: track 48.6 -> 50.9 mm, vias 1 -> 2
- net RESET: track 39.6 -> 38.2 mm
- net GND: track 53.2 -> 54.0 mm, vias 13 -> 15
